File: bkm-10rlternative.kicad_pcb (KiCad board)
At the start: 4 copper layers, 210.8 x 74.9 mm, 257 parts, among them J1 DB9_Male_MountingHoles, J2 ICSP, Q1 MMBT3904, Q10 MMBT3904, Q11 MMBT3904, Q12 MMBT3904, Q13 MMBT3904, Q14 MMBT3904, Q2 MMBT3904, Q3 MMBT3904, Q4 MMBT3904, Q5 MMBT3904, Q6 MMBT3904, Q7 MMBT3904, Q8 MMBT3904, Q9 MMBT3904, SW1 SHIFT, SW10 ADDR_SAFE_AREA, SW11 UP, SW12 MENU, SW13 DOWN, SW14 ENTER, SW15 DEGAUSS, SW16 POWER, SW17 KEY_1, SW18 KEY_2, SW19 KEY_3, SW2 HORIZ_SYNC, SW20 KEY_4, SW21 KEY_5, SW22 KEY_6, SW23 KEY_7, SW24 KEY_8, SW25 KEY_9, SW26 KEY_DEL, SW27 KEY_0, SW28 KEY_ENTER, SW29 CONTRAST_MANUAL, SW3 UNDERSCAN_16_9, SW30 CONTRAST_KNOB, SW31 BRIGHT_MANUAL, SW32 BRIGHT_KNOB, SW33 CHROMA_MANUAL, SW34 CHROMA_KNOB, SW35 PHASE_MANUAL, SW36 PHASE_KNOB, SW4 VERT_BLUE_ONLY, SW5 MONO_R, SW6 APT_G, SW7 COMB_B, SW8 F1_F3, SW9 F2_F4, U1 74LVC2G14, U10 MCP23S17_SS, U11 MCP23S17_SS, U12 MCP23S17_SS, U13 74LVC2G14, U14 74LVC2G14, U15 74LVC2G14, U16 74LVC2G14, U17 74LVC2G14, U18 74LVC2G14, U19 74LVC2G14, U2 74HC14, U20 74LVC2G14, U3 74HC14, U4 74HC14, U5 74HC14, U6 TSOP382xx, U8 MAX491E, U9 ATmega328PB-AU, Y1 Resonator

Commit message: Initial revision B
Parts:
- removed Q10, Q2, Q3, Q4, Q5, Q6, Q7, Q8, Q9: MMBT3904, Package_TO_SOT_SMD:SOT-23
- removed R102, R103, R104, R105, R106, R107, R108, R109, R110: 560R, Resistor_SMD:R_0603_1608Metric_Pad0.98x0.95mm_HandSolder
- removed R111, R113, R115: 1K, Resistor_SMD:R_0603_1608Metric_Pad0.98x0.95mm_HandSolder
- removed R99: 10K, Resistor_SMD:R_0603_1608Metric_Pad0.98x0.95mm_HandSolder
- added C56: 10uF, Capacitor_SMD:C_0805_2012Metric_Pad1.18x1.45mm_HandSolder, F.Cu at (66.0, 100.0)
- added C57: 10uF, Capacitor_SMD:C_0805_2012Metric_Pad1.18x1.45mm_HandSolder, F.Cu at (65.9, 104.5)
- added C58: 100nF, Capacitor_SMD:C_0603_1608Metric_Pad1.08x0.95mm_HandSolder, F.Cu at (66.0, 102.2)
- added C59: 100nF, Capacitor_SMD:C_0603_1608Metric_Pad1.08x0.95mm_HandSolder, F.Cu at (62.0, 91.8)
- added J3: Micro_SD_Card_Det, MEM2061:MEM2061, F.Cu at (60.3, 78.4)
- added J4: Conn_01x05_Male, Connector_PinHeader_2.54mm:PinHeader_1x05_P2.54mm_Vertical, F.Cu at (239.1, 84.5)
- added U201: 74LVC2G34, Package_TO_SOT_SMD:SOT-23-6_Handsoldering, F.Cu at (207.1, 84.0)
- added U202: 74LVC2G34, Package_TO_SOT_SMD:SOT-23-6_Handsoldering, F.Cu at (195.4, 84.0)
- added U203: 74LVC2G34, Package_TO_SOT_SMD:SOT-23-6_Handsoldering, F.Cu at (184.0, 84.0)
- added U204: 74LVC2G34, Package_TO_SOT_SMD:SOT-23-6_Handsoldering, F.Cu at (172.6, 84.0)
- added U205: 74LVC2G34, Package_TO_SOT_SMD:SOT-23-6_Handsoldering, F.Cu at (161.2, 84.0)
- added U206: 74LVC2G34, Package_TO_SOT_SMD:SOT-23-6_Handsoldering, F.Cu at (149.6, 84.0)
- added U207: 74LVC2G34, Package_TO_SOT_SMD:SOT-23-6_Handsoldering, F.Cu at (138.3, 84.0)
- added U208: 74LVC2G34, Package_TO_SOT_SMD:SOT-23-6_Handsoldering, F.Cu at (126.7, 84.0)
- added U209: 74LVC2G34, Package_TO_SOT_SMD:SOT-23-6_Handsoldering, F.Cu at (115.5, 84.0)
- added U21: NCP1117-3.3_SOT223, Package_TO_SOT_SMD:SOT-223-3_TabPin2, F.Cu at (59.5, 102.2)
- added U22: 74LVC125, Package_SO:TSSOP-14_4.4x5mm_P0.65mm, F.Cu at (65.7, 93.8)
- R53: value NM -> 1K
- SW1, SW10, SW2, SW29, SW3, SW31, SW33, SW35, SW4, SW5, SW6, SW7, SW8, SW9: footprint TL-1240:TL-1240 -> TL-1265:TL-1265
- SW11, SW12, SW13, SW14, SW15, SW16, SW17, SW18, SW19, SW20, SW21, SW22, SW23, SW24, SW25, SW26, SW27, SW28: footprint TL-1240:TL-1240 -> TL-1265:TL-1265_NO_LED
- U2, U3, U4, U5: footprint Package_SO:SSOP-14_5.3x6.2mm_P0.65mm -> Package_SO:TSSOP-14_4.4x5mm_P0.65mm
- moved R53 166.8 mm to (71.9, 96.2), turned to 90 degrees
- moved R98 29.9 mm to (62.4, 87.0), turned to 270 degrees
- moved U6 28.1 mm to (46.3, 56.8)
- moved C8 13.8 mm to (76.5, 101.9), turned to 0 degrees
- moved R90 11.7 mm to (193.8, 65.5), turned to 270 degrees
- moved R80 11.6 mm to (144.0, 89.3)
- moved R93 11.6 mm to (182.7, 65.5), turned to 270 degrees
- moved R78 11.6 mm to (166.9, 89.4)
- moved R77 11.5 mm to (178.4, 89.4)
- moved R81 11.4 mm to (132.7, 89.0)
- moved R75 11.4 mm to (189.9, 89.4)
- moved R79 11.4 mm to (155.5, 89.4)
- moved R82 11.4 mm to (121.3, 89.1)
- moved R74 11.3 mm to (212.6, 89.4)
- moved R76 11.3 mm to (201.3, 89.4)
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Connections:
- J2 pad 1: CHROMA_A -> ICSP_MISO
- J2 pad 3: CHROMA_B -> ICSP_SCK
- J2 pad 4: BRIGHT_B -> ICSP_MOSI
- R53 pad 1: /MCU+RS485/RXD -> Net-(R53-Pad1)
- R53 pad 2: /MCU+RS485/~RXD -> ICSP_MISO
- R55 pad 2: GND -> Net-(R55-Pad2)
- R56 pad 2: GND -> Net-(R56-Pad2)
- R57 pad 2: GND -> Net-(R57-Pad2)
- R58 pad 2: GND -> Net-(R58-Pad2)
- R59 pad 2: GND -> Net-(R59-Pad2)
- R60 pad 2: GND -> Net-(R60-Pad2)
- R61 pad 2: GND -> Net-(R61-Pad2)
- R62 pad 2: GND -> Net-(R62-Pad2)
- R63 pad 2: GND -> Net-(R63-Pad2)
- R98 pad 1: SS1 -> SD_CARD_DET
- SW11 pad 4: (no net) -> Net-(SW11-Pad4)
- SW12 pad 4: (no net) -> Net-(SW12-Pad4)
- SW13 pad 4: (no net) -> Net-(SW13-Pad4)
- SW14 pad 4: (no net) -> Net-(SW14-Pad4)
- SW15 pad 4: (no net) -> Net-(SW15-Pad4)
- SW16 pad 4: (no net) -> Net-(SW16-Pad4)
- SW29 pad 4: (no net) -> Net-(SW29-Pad4)
- SW31 pad 4: (no net) -> Net-(SW31-Pad4)
- SW33 pad 4: (no net) -> Net-(SW33-Pad4)
- SW35 pad 4: (no net) -> Net-(SW35-Pad4)
- U10 pad 11: SS2 -> SS0
- U10 pad 19: (no net) -> Net-(U10-Pad19)
- U10 pad 20: (no net) -> Net-(U10-Pad20)
- U10 pad 27: (no net) -> Net-(U10-Pad27)
- U10 pad 28: (no net) -> Net-(U10-Pad28)
- U11 pad 1: (no net) -> DOWN_SW_IN
- U11 pad 19: (no net) -> Net-(U11-Pad19)
- U11 pad 2: (no net) -> ENTER_SW_IN
- U11 pad 20: (no net) -> Net-(U11-Pad20)
- U11 pad 25: (no net) -> UP_SW_IN
- U11 pad 26: (no net) -> MENU_SW_IN
- U12 pad 11: SS1 -> SS0
- U12 pad 19: (no net) -> Net-(U12-Pad19)
- U12 pad 20: (no net) -> Net-(U12-Pad20)
- U17 pad 4: Net-(R111-Pad2) -> BRIGHT_B
- U18 pad 4: Net-(R113-Pad2) -> CHROMA_B
- U18 pad 6: Net-(R115-Pad2) -> CHROMA_A
- U3 pad 10: (no net) -> Net-(U3-Pad10)
- U3 pad 8: (no net) -> Net-(U3-Pad8)
- U8 pad 1: (no net) -> Net-(U8-Pad1)
- U8 pad 13: (no net) -> Net-(U8-Pad13)
- U8 pad 3: UART_CTS -> GND
- U8 pad 4: UART_RTS -> VCC
- U8 pad 8: (no net) -> Net-(U8-Pad8)
- U9 pad 1: UART_CTS -> PHASE_B
- U9 pad 10: ENTER_SW_IN -> BRIGHT_A
- U9 pad 11: DOWN_SW_IN -> SD_CARD_DET
- U9 pad 14: BRIGHT_A -> SD_SS
- U9 pad 15: BRIGHT_B -> ICSP_MOSI
- U9 pad 16: CHROMA_A -> ICSP_MISO
- U9 pad 17: CHROMA_B -> ICSP_SCK
- U9 pad 19: PHASE_B -> Net-(U9-Pad19)
- U9 pad 2: UP_SW_IN -> Net-(U9-Pad2)
- U9 pad 25: SS2 -> SS0
- U9 pad 26: SS1 -> CHROMA_A
- U9 pad 27: SS0 -> CHROMA_B
- U9 pad 32: UART_RTS -> PHASE_A
- U9 pad 6: PHASE_A -> Net-(U9-Pad6)
- U9 pad 9: MENU_SW_IN -> BRIGHT_B
Routing:
- net UART_CTS: track 169.4 -> 0.00 mm, vias 2 -> 0
- net UART_RTS: track 167.4 -> 0.00 mm, vias 2 -> 0
- net SS1: track 134.9 -> 0.00 mm, vias 2 -> 0
- net SHIFT_ACTIVE_LED: track 134.7 -> 256.1 mm, vias 0 -> 10
- net SS0: track 35.3 -> 153.8 mm, vias 0 -> 2
- net +3V3: track 0.00 -> 44.3 mm, vias 0 -> 3
- net ICSP_MOSI: track 0.00 -> 40.3 mm, vias 0 -> 2
- net ICSP_MISO: track 0.00 -> 36.5 mm, vias 0 -> 2
- net ICSP_SCK: track 0.00 -> 33.3 mm
- net GND: track 83.0 -> 114.4 mm, vias 68 -> 87
- net SD_MISO_LV: track 0.00 -> 30.3 mm
- net SS2: track 28.2 -> 0.00 mm
- net SD_MOSI_LV: track 0.00 -> 24.8 mm
- net SD_SCK_LV: track 0.00 -> 23.5 mm, vias 0 -> 2
- net DOWN_SW_IN: track 30.1 -> 53.2 mm, vias 0 -> 2
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Other:
- board text added: "GND"
- board text added: "RXD"
- board text added: "Rev. B"
- board text added: "TXD"
- board text added: "~RXD"
- board text added: "~TXD"
- board text removed: "Rev. A"
